Commit message: Retargeting works now for bitbots pi_plus

File: source/whole_body_tracking/whole_body_tracking/assets/hightorque/pi_plus_bitbots/pi_plus_22dof.urdf (robot description, URDF)
Before this commit: robot PiPlus_S_12L8A0G2H0W, 32 links, 31 joints
Joints:
- joint head_pitch_joint: axis 0 1 0 -> (none); limit lower=-1.23 upper=1.01 effort=3 velocity=30.37 -> (none); type revolute -> fixed
- joint head_yaw_joint: axis 0 0 1 -> (none); limit lower=-1.43 upper=1.43 effort=3 velocity=30.37 -> (none); type revolute -> fixed
- joint l_calf_joint: axis 0 -1 0 -> 0 1 0; limit lower=-2.26 upper=2.14 effort=20 velocity=5.45 -> lower=-2.14 upper=2.26 effort=20 velocity=5.45
- joint l_thigh_joint: axis 0 0 -1 -> 0 0 1; limit lower=-2.82 upper=2.49 effort=20 velocity=5.45 -> lower=-2.49 upper=2.82 effort=20 velocity=5.45
- joint l_upper_arm_joint: axis 0 0 -1 -> 0 0 1
- joint r_ankle_pitch_joint: axis 0 -1 0 -> 0 1 0; limit lower=-1 upper=0.87 effort=20 velocity=5.45 -> lower=-0.87 upper=1 effort=20 velocity=5.45
- joint r_elbow_joint: axis 0 -1 0 -> 0 1 0; limit lower=-1.86 upper=2.1 effort=10 velocity=15.91 -> lower=-2.1 upper=1.86 effort=10 velocity=15.91
- joint r_hip_pitch_joint: axis 0 -1 0 -> 0 1 0
- joint r_shoulder_pitch_joint: axis 0 -1 0 -> 0 1 0
- joint r_thigh_joint: axis 0 0 -1 -> 0 0 1; limit lower=-2.82 upper=2.49 effort=20 velocity=5.45 -> lower=-2.49 upper=2.82 effort=20 velocity=5.45
- joint r_upper_arm_joint: axis 0 0 -1 -> 0 0 1

Commit message: added proper punishing of undesired contacts

File: source/whole_body_tracking/whole_body_tracking/assets/hightorque/pi_plus_bitbots/pi_plus_22dof.urdf (robot description, URDF)
Before this commit: robot PiPlus_S_12L8A0G2H0W, 32 links, 31 joints
Links:
- removed link camera_link
- removed link camera_optical_frame_right_uncalibrated
- removed link camera_optical_frame_uncalibrated
- removed link imu_frame_uncalibrated
- removed link l_sole
- removed link r_sole
Joints:
- removed joint camera_joint
- removed joint camera_joint_right_uncalibrated
- removed joint camera_joint_uncalibrated
- removed joint imu_frame_joint
- removed joint l_sole_joint
- removed joint r_sole_joint

Commit message: improved retargeting pipeline

File: source/whole_body_tracking/whole_body_tracking/assets/hightorque/pi_plus_bitbots/pi_plus_22dof.urdf (robot description, URDF)
Before this commit: robot PiPlus_S_12L8A0G2H0W, 26 links, 25 joints
Joints:
- joint l_ankle_pitch_joint: limit lower=-0.87 upper=1 effort=20 velocity=5.45 -> lower=-0.85 upper=0.95 effort=20 velocity=5.45
- joint l_ankle_roll_joint: limit lower=-0.78 upper=0.78 effort=20 velocity=5.45 -> lower=-0.72 upper=0.72 effort=20 velocity=5.45
- joint l_calf_joint: axis 0 1 0 -> 0 -1 0; limit lower=-2.14 upper=2.26 effort=20 velocity=5.45 -> lower=-2.21 upper=1.97 effort=20 velocity=5.45
- joint l_elbow_joint: limit lower=-2.1 upper=1.86 effort=10 velocity=15.91 -> lower=-2.04 upper=1.8 effort=10 velocity=15.91
- joint l_hip_pitch_joint: limit lower=-2.89 upper=2.89 effort=20 velocity=5.45 -> lower=-2.84 upper=2.84 effort=20 velocity=5.45
- joint l_hip_roll_joint: limit lower=-0.2 upper=3.14 effort=20 velocity=5.45 -> lower=-0.15 upper=3.1 effort=20 velocity=5.45
- joint l_shoulder_pitch_joint: limit lower=-2.6 upper=2.6 effort=10 velocity=15.91 -> lower=-2.55 upper=2.55 effort=10 velocity=15.91
- joint l_shoulder_roll_joint: limit lower=-1.46 upper=1.65 effort=10 velocity=15.91 -> lower=-1.4 upper=1.65 effort=10 velocity=15.91
- joint l_thigh_joint: axis 0 0 1 -> 0 0 -1; limit lower=-2.49 upper=2.82 effort=20 velocity=5.45 -> lower=-2.77 upper=2.45 effort=20 velocity=5.45
- joint l_upper_arm_joint: axis 0 0 1 -> 0 0 -1; limit lower=-2.6 upper=2.6 effort=10 velocity=15.91 -> lower=-2.55 upper=2.55 effort=10 velocity=15.91
- joint r_ankle_pitch_joint: axis 0 1 0 -> 0 -1 0; limit lower=-0.87 upper=1 effort=20 velocity=5.45 -> lower=-0.95 upper=0.85 effort=20 velocity=5.45
- joint r_ankle_roll_joint: limit lower=-0.78 upper=0.78 effort=20 velocity=5.45 -> lower=-0.72 upper=0.72 effort=20 velocity=5.45
- joint r_calf_joint: limit lower=-2.14 upper=2.26 effort=20 velocity=5.45 -> lower=-1.97 upper=2.21 effort=20 velocity=5.45
- joint r_elbow_joint: axis 0 1 0 -> 0 -1 0; limit lower=-2.1 upper=1.86 effort=10 velocity=15.91 -> lower=-1.8 upper=2.04 effort=10 velocity=15.91
- joint r_hip_pitch_joint: axis 0 1 0 -> 0 -1 0; limit lower=-2.89 upper=2.89 effort=20 velocity=5.45 -> lower=-2.84 upper=2.84 effort=20 velocity=5.45
- joint r_hip_roll_joint: limit lower=-3.14 upper=0.2 effort=20 velocity=5.45 -> lower=-3.1 upper=0.15 effort=20 velocity=5.45
- joint r_shoulder_pitch_joint: axis 0 1 0 -> 0 -1 0; limit lower=-2.6 upper=2.6 effort=10 velocity=15.91 -> lower=-2.55 upper=2.55 effort=10 velocity=15.91
- joint r_shoulder_roll_joint: limit lower=-1.65 upper=1.46 effort=10 velocity=15.91 -> lower=-1.65 upper=1.4 effort=10 velocity=15.91
- joint r_thigh_joint: axis 0 0 1 -> 0 0 -1; limit lower=-2.49 upper=2.82 effort=20 velocity=5.45 -> lower=-2.77 upper=2.45 effort=20 velocity=5.45
- joint r_upper_arm_joint: axis 0 0 1 -> 0 0 -1; limit lower=-2.6 upper=2.6 effort=10 velocity=15.91 -> lower=-2.55 upper=2.55 effort=10 velocity=15.91

Commit message: limit knee joint in urdf

File: source/whole_body_tracking/whole_body_tracking/assets/hightorque/pi_plus_bitbots/pi_plus_22dof.urdf (robot description, URDF)
Before this commit: robot PiPlus_S_12L8A0G2H0W, 26 links, 25 joints
Joints:
- joint l_calf_joint: limit lower=-2.21 upper=1.97 effort=20 velocity=5.45 -> lower=-2.21 upper=0.05 effort=20 velocity=5.45
- joint r_calf_joint: limit lower=-1.97 upper=2.21 effort=20 velocity=5.45 -> lower=-0.05 upper=2.21 effort=20 velocity=5.45

Commit message: fix sim2sim validation script

File: source/whole_body_tracking/whole_body_tracking/assets/hightorque/pi_plus_bitbots/pi_plus_22dof.urdf (robot description, URDF)
Before this commit: robot PiPlus_S_12L8A0G2H0W, 26 links, 25 joints
Joints:
- joint l_calf_joint: limit lower=-2.21 upper=0.05 effort=20 velocity=5.45 -> lower=-2.21 upper=0.1 effort=20 velocity=5.45
- joint r_calf_joint: limit lower=-0.05 upper=2.21 effort=20 velocity=5.45 -> lower=-0.1 upper=2.21 effort=20 velocity=5.45
